File: hw/rack/out/sch/backplane_rf_a1.kicad_sch (KiCad schematic)
At the start: 48 parts, among them J3 ANT A, U10 TPS259541DSGR, U6 QPL9057, U8 QPQ1907

Commit message: hw/rack: #95 review fixes: QPQ1907 pinout + RF continuity test, 1 ohm 2512 bias-T, input fuse, keyed slots, CM4 source, CI scikit-rf + stale check, ADR-0018 gain-plan stop-and-ask (#33)
- QPQ1907 pins per datasheet 040820 (1 in, 4 out, 2/3/5 GND); test walks BNC to every slot port
- bias-T 1 ohm 2512 (0.27 W at 0.52 A), resistor power ratings asserted
- 4 A fuse ahead of the TVS; Harwin M20-7831346 + M20-003 key at position 14
- CM4002008 from The Pi Hut (GBP 79.20); Lite-On LEDs
- Wilkinson +-10 % width sweep; netlist timestamp stripped
- CI: scikit-rf installed, cross-check required under CI, hw/rack stale-output diff
- Audit 6: per-carrier NF, stage headroom at 0.5/1/1.5 m (wings), phones, nRF5340 PS v1.1
  C/I + PIMD, nRF21540 P1dB; no fixed gain plan meets both: stop-and-ask

Co-Authored-By: Claude Opus 5.5 <noreply@anthropic.com>
Parts:
- R17: value 10 -> 1; footprint Resistor_SMD:R_0402_1005Metric -> Resistor_SMD:R_2512_6332Metric; MPN R_0402_1% -> R_2512_1R_1W; P_W (none) -> 1.0
- R18, R19, R20, R21, R22, R23, R24, R25, R26, R27, R28, R29: P_W (none) -> 0.0625
- U8: footprint openpack:Qorvo_QPQ1907_1.4x1.2mm -> openpack:Qorvo_QPQ1907_LGA5_1.4x1.2mm_datasheet_land_pattern
Connections:
- net WK_A_10a is gone; now on net SPL_A_IN: R23.1, R25.2, R26.1, R27.2, R28.2, TL1.2, TL10.2, TL12.2, TL13.1, TL14.1, TL3.1, TL4.1, TL6.2, TL7.2
- net WK_A_10b is gone; now on net SPL_A_IN: R23.2, R24.2, R26.2, R28.1, TL10.1, TL11.2, TL2.2, TL4.2, TL5.1, TL6.1, TL8.2, TL9.1
- net GND: now also R21.2, U6.2 (RF_IN), U8.3 (GND3); no longer U8.4 (GND4)
- net SPL_A_IN: now also R24.1, TL3.2, TL7.1, TL8.1, U8.4 (RF_OUT); no longer U8.3 (RF_OUT)
Other:
- moved on the sheet: C28, C29, C30, C31, C32, C33, C34, C35, C36, C37, C38, D1_1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
