File: hw/rack/out/sch/backplane_rf_b1.kicad_sch (KiCad schematic)
At the start: 48 parts, among them J4 ANT B, U11 TPS259541DSGR, U7 QPL9057, U9 QPQ1907

Commit message: hw/rack: #95 review fixes: QPQ1907 pinout + RF continuity test, 1 ohm 2512 bias-T, input fuse, keyed slots, CM4 source, CI scikit-rf + stale check, ADR-0018 gain-plan stop-and-ask (#33)
- QPQ1907 pins per datasheet 040820 (1 in, 4 out, 2/3/5 GND); test walks BNC to every slot port
- bias-T 1 ohm 2512 (0.27 W at 0.52 A), resistor power ratings asserted
- 4 A fuse ahead of the TVS; Harwin M20-7831346 + M20-003 key at position 14
- CM4002008 from The Pi Hut (GBP 79.20); Lite-On LEDs
- Wilkinson +-10 % width sweep; netlist timestamp stripped
- CI: scikit-rf installed, cross-check required under CI, hw/rack stale-output diff
- Audit 6: per-carrier NF, stage headroom at 0.5/1/1.5 m (wings), phones, nRF5340 PS v1.1
  C/I + PIMD, nRF21540 P1dB; no fixed gain plan meets both: stop-and-ask

Co-Authored-By: Claude Opus 5.5 <noreply@anthropic.com>
Parts:
- R30: value 10 -> 1; footprint Resistor_SMD:R_0402_1005Metric -> Resistor_SMD:R_2512_6332Metric; MPN R_0402_1% -> R_2512_1R_1W; P_W (none) -> 1.0
- R31, R32, R33, R34, R35, R36, R37, R38, R39, R40, R41, R42: P_W (none) -> 0.0625
- U9: footprint openpack:Qorvo_QPQ1907_1.4x1.2mm -> openpack:Qorvo_QPQ1907_LGA5_1.4x1.2mm_datasheet_land_pattern
Connections:
- net WK_B_10a is gone; now on net SPL_B_IN: R36.1, R38.2, R39.1, R40.1, R41.2, TL15.2, TL17.1, TL18.1, TL20.2, TL21.2, TL23.2, TL26.2, TL27.1, TL28.1
- net WK_B_10b is gone; now on net SPL_B_IN: R36.2, R37.2, R39.2, R41.1, TL16.2, TL18.2, TL19.1, TL20.1, TL22.2, TL23.1, TL24.1, TL25.2
- net GND: now also R34.2, U7.2 (RF_IN), U9.3 (GND3); no longer U9.4 (GND4)
- net SPL_B_IN: now also R37.1, TL17.2, TL21.1, TL22.1, U9.4 (RF_OUT); no longer U9.3 (RF_OUT)
Other:
- moved on the sheet: C39, C40, C41, C42, C43, C44, C45, C46, C47, C48, C49, D4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
