File: hw/rack/out/sch/backplane_slots1.kicad_sch (KiCad schematic)
At the start: 200 parts, among them J10 SLOT 0, J11 SLOT 1, J12 SLOT 2, J13 SLOT 3, J14 SLOT 4, J15 SLOT 5, J16 SLOT 6, J17 SLOT 7, J20 OUT 1, J21 OUT 2, J22 OUT 3, J23 OUT 4, J24 OUT 5, J25 OUT 6, J26 OUT 7, J27 OUT 8, J30 RF A0, J31 RF A1, J32 RF A2, J33 RF A3, J34 RF A4, J35 RF A5, J36 RF A6, J37 RF A7, J40 RF B0, J41 RF B1, J42 RF B2, J43 RF B3, J44 RF B4, J45 RF B5, J46 RF B6, J47 RF B7, U20 TPS259541DSGR, U21 TPS259541DSGR, U22 TPS259541DSGR, U23 TPS259541DSGR, U24 TPS259541DSGR, U25 TPS259541DSGR, U26 TPS259541DSGR, U27 TPS259541DSGR, U30 TPS259531DSGR, U31 TPS259531DSGR, U32 TPS259531DSGR, U33 TPS259531DSGR, U34 TPS259531DSGR, U35 TPS259531DSGR, U36 TPS259531DSGR, U37 TPS259531DSGR

Commit message: hw/rack: #95 review fixes: QPQ1907 pinout + RF continuity test, 1 ohm 2512 bias-T, input fuse, keyed slots, CM4 source, CI scikit-rf + stale check, ADR-0018 gain-plan stop-and-ask (#33)
- QPQ1907 pins per datasheet 040820 (1 in, 4 out, 2/3/5 GND); test walks BNC to every slot port
- bias-T 1 ohm 2512 (0.27 W at 0.52 A), resistor power ratings asserted
- 4 A fuse ahead of the TVS; Harwin M20-7831346 + M20-003 key at position 14
- CM4002008 from The Pi Hut (GBP 79.20); Lite-On LEDs
- Wilkinson +-10 % width sweep; netlist timestamp stripped
- CI: scikit-rf installed, cross-check required under CI, hw/rack stale-output diff
- Audit 6: per-carrier NF, stage headroom at 0.5/1/1.5 m (wings), phones, nRF5340 PS v1.1
  C/I + PIMD, nRF21540 P1dB; no fixed gain plan meets both: stop-and-ask

Co-Authored-By: Claude Opus 5.5 <noreply@anthropic.com>
Parts:
- D11, D15, D19, D23, D27, D31, D35, D7: MPN LED_0603_GREEN -> LTST-C191KGKT
- D12, D16, D20, D24, D28, D32, D36, D8: MPN LED_0603_RED -> LTST-C191KRKT
- J10, J11, J12, J13, J14, J15, J16, J17: MPN PPPC132LFBN-RC -> M20-7831346
- R43, R44, R45, R46, R47, R48, R49, R50, R51, R52, R53, R54, R55, R56, R57, R58, R59, R60, R61, R62, R63, R64, R65, R66, R67, R68, R69, R70, R71, R72, R73, R74, R75, R76, R77, R78, R79, R80, R81, R82, R83, R84, R85, R86, R87, R88, R89, R90, R91, R92, R93, R94, R95, R96, R97, R98: P_W (none) -> 0.0625
Other:
- moved on the sheet: C50, C51, C52, C53, C54, C55, C56, C57, C58, C59, C60, C61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
