File: hw/pack/out/sch/pack_mcu_usb1.kicad_sch (KiCad schematic)
At the start: 23 parts, among them J2 USB-C, J3 SWD, U1 BT40NE, U7 USBLC6-2SC6

Commit message: pack: cost-down to PK-12 $33.34: printed cell cradle + MYOUNG contacts, LCSC IPEX pigtail, priced M2 screws (#34)
- BT1: MYOUNG MY-18650-04-J/-05-J (LCSC C19184125/C19184124) in a printed
  cradle in the base (76 mm plate faces: spring 4.2-9.2 mm for 70-65 mm cells);
  the SMT BH-18650-B1BA002 holder is gone; footprint Cell_Wire_Pads
- pigtail: BAT Wireless BWIPX1-SMA-1.13L150 (LCSC C784404, $0.6015 @100), SMA
  cut off, ~100 mm + 31 mm wire whip; audit.py PIGTAIL_IL 0.46 <= 0.6 dB
- audit.py cutoff path includes the spring (0.10 ohm), cutoff stays 3.2 V
- 2 x M2x6 PT screws $0.112 (Fastener Superstore 585907)
- prices.py, bom.csv, pack_uk.csv (UK $34.81) updated

Co-Authored-By: Claude Opus 5.5 <noreply@anthropic.com>
Other:
- moved on the sheet: C28, C29, C30, C31, C32, D1, D2, D3, D4, J2, J3, R12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
