File: hw/rack/rack.kicad_pcb (KiCad board)
At the start: 4 copper layers, 412 x 323 mm, 444 parts, among them J1 12V IN, J10 SLOT 0, J11 SLOT 1, J12 SLOT 2, J13 SLOT 3, J14 SLOT 4, J15 SLOT 5, J16 SLOT 6, J17 SLOT 7, J2 CM4IO J8, J20 OUT 1, J21 OUT 2, J22 OUT 3, J23 OUT 4, J24 OUT 5, J25 OUT 6, J26 OUT 7, J27 OUT 8, J3 ANT A, J30 RF A0, J31 RF A1, J32 RF A2, J33 RF A3, J34 RF A4, J35 RF A5, J36 RF A6, J37 RF A7, J4 ANT B, J40 RF B0, J41 RF B1, J42 RF B2, J43 RF B3, J44 RF B4, J45 RF B5, J46 RF B6, J47 RF B7, J5 CM4IO 12V, Q1 AO4407A, U1 TPS259541DSGR, U10 TPS259541DSGR, U11 TPS259541DSGR, U12 TPS259541DSGR, U2 TPS62933DRLR, U20 TPS259541DSGR, U21 TPS259541DSGR, U22 TPS259541DSGR, U23 TPS259541DSGR, U24 TPS259541DSGR, U25 TPS259541DSGR, U26 TPS259541DSGR, U27 TPS259541DSGR, U3 TLV76733, U30 TPS259531DSGR, U31 TPS259531DSGR, U32 TPS259531DSGR, U33 TPS259531DSGR, U34 TPS259531DSGR, U35 TPS259531DSGR, U36 TPS259531DSGR, U37 TPS259531DSGR, U4 SC16IS752IPW, U5 SC16IS752IPW, U6 QPL9057, U7 QPL9057, U8 QPQ1907, U9 QPQ1907, Y1 14.7456M, Y2 14.7456M

Commit message: hw/rack: #126 review fixes: Wilkinson limit 14 dB (SPEC RK-5, ADR-0018 with history), PCB order £300 est., board 321.5 mm deep (2.35 mm front gap, LED check), HCI 60 ohm -40..85 C crystal + 33 pF, RK-2 on the NF need, power note, stale text, dangling stubs pruned (#34)
Co-Authored-By: Claude Opus 5.5 <noreply@anthropic.com>
Parts:
- C21, C22, C25, C26: value 22p -> 33p
- TL1, TL10, TL11, TL12, TL13, TL14, TL15, TL16, TL17, TL18, TL19, TL2, TL20, TL21, TL22, TL23, TL24, TL25, TL26, TL27, TL28, TL3, TL4, TL5, TL6, TL7, TL8, TL9: value 70R7 L/4 17.76mm w0.196 -> 70R7 L/4 18.02mm w0.170
- moved D10 1.50 mm to (130.0, -220.2)
- moved D13 1.50 mm to (170.0, -220.2)
- moved D14 1.50 mm to (182.0, -220.2)
- moved D17 1.50 mm to (222.0, -220.2)
- moved D18 1.50 mm to (234.0, -220.2)
- moved D21 1.50 mm to (274.0, -220.2)
- moved D22 1.50 mm to (286.0, -220.2)
- moved D25 1.50 mm to (326.0, -220.2)
- moved D26 1.50 mm to (338.0, -220.2)
- moved D29 1.50 mm to (378.0, -220.2)
- moved D30 1.50 mm to (390.0, -220.2)
- moved D33 1.50 mm to (430.0, -220.2)
- moved D34 1.50 mm to (442.0, -220.2)
- moved D37 1.50 mm to (482.0, -220.2)
- moved D38 1.50 mm to (494.0, -220.2)
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Routing:
- net S1_BP_BOOT: track 120.3 -> 117.9 mm
- net S0_BP_BOOT: track 167.9 -> 165.5 mm
- net S4_BP_BOOT: track 71.0 -> 68.7 mm
- net HOST_GPIO25: track 133.8 -> 131.5 mm
- net S4_BP_LED_PEAK: track 172.9 -> 171.4 mm
- net S1_BP_LED_PEAK: track 172.5 -> 171.0 mm
- net S4_BP_LED_LOCK: track 178.3 -> 176.8 mm
- net S6_BP_LED_LOCK: track 167.3 -> 165.8 mm
- net S5_BP_LED_LOCK: track 167.3 -> 165.8 mm
- net S7_BP_LED_LOCK: track 167.3 -> 165.8 mm
- net S1_BP_LED_LOCK: track 165.3 -> 163.8 mm
- net S3_BP_LED_LOCK: track 168.8 -> 167.3 mm
- net S2_BP_LED_LOCK: track 165.3 -> 163.8 mm
- net S0_BP_LED_LOCK: track 165.4 -> 163.9 mm
- net S0_BP_LED_PEAK: track 164.7 -> 163.2 mm
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Other:
- board size 412 x 323 mm -> 412 x 321.5 mm
